Commit message: IMU integrada y probada en el portátil: nodo imu_bmi160.py sin instalar nada, imu_link en la URDF, imu:=true con EKF (avance de rf2o, rumbo de la IMU) y margen_llegada en el lanzador; IMU= y MARGEN= en nav2_mapa_guardado.sh

File: Robot/aws-deepracer/deepracer_description/models/urdf/deepracer_hardware.urdf (robot description, URDF)
Before this commit: robot deepracer_hardware, 3 links, 2 joints
Links:
- added link imu_link
Joints:
- added joint imu_joint: type fixed, parent base_link, child imu_link, origin xyz=0 0 0 rpy=3.1416 0 1.5708
